File: Code_And_Circuits/Full_Circuit/Full_Circuit.kicad_pcb (KiCad board)
At the start: 2 copper layers, 0 parts

Commit message: Reconfired some pin assignments for cleaner layout and adding reference footprints and mostly layed out board, due to space limits logging section has been ommitted
Parts:
- added A1: Arduino_Nano_ESP32, Module:Arduino_Nano, B.Cu at (135.4, 61.6)
- added C1: 1000PF, Capacitor_SMD:C_0805_2012Metric_Pad1.18x1.45mm_HandSolder, F.Cu at (126.6, 60.6)
- added C10: 1uF, Capacitor_SMD:C_0805_2012Metric_Pad1.18x1.45mm_HandSolder, B.Cu at (152.0, 121.0)
- added C11: 1uF, Capacitor_SMD:C_0805_2012Metric_Pad1.18x1.45mm_HandSolder, B.Cu at (154.2, 121.0)
- added C12: 1uF, Capacitor_SMD:C_0805_2012Metric_Pad1.18x1.45mm_HandSolder, B.Cu at (156.5, 120.9)
- added C13: 1uF, Capacitor_SMD:C_0805_2012Metric_Pad1.18x1.45mm_HandSolder, B.Cu at (156.7, 131.4)
- added C14: 1uF, Capacitor_SMD:C_0805_2012Metric_Pad1.18x1.45mm_HandSolder, B.Cu at (159.6, 126.7)
- added C15: 1uF, Capacitor_SMD:C_0805_2012Metric_Pad1.18x1.45mm_HandSolder, B.Cu at (162.2, 121.1)
- added C17: 10 uF, Capacitor_THT:C_Disc_D3.0mm_W1.6mm_P2.50mm, F.Cu at (211.2, 78.2)
- added C18: 10 uF, Capacitor_THT:C_Disc_D3.0mm_W1.6mm_P2.50mm, F.Cu at (174.5, 55.6)
- added C5: 1000PF, Capacitor_SMD:C_0805_2012Metric_Pad1.18x1.45mm_HandSolder, F.Cu at (132.2, 70.7)
- added C6: 0.1 uF, Capacitor_SMD:C_0805_2012Metric_Pad1.18x1.45mm_HandSolder, F.Cu at (179.8, 77.0)
- added C7: 0.33uF, Capacitor_SMD:C_0805_2012Metric_Pad1.18x1.45mm_HandSolder, F.Cu at (185.3, 77.0)
- added C8: 1uF, Capacitor_SMD:C_0805_2012Metric_Pad1.18x1.45mm_HandSolder, B.Cu at (147.3, 121.0)
- added C9: 1uF, Capacitor_SMD:C_0805_2012Metric_Pad1.18x1.45mm_HandSolder, B.Cu at (149.6, 121.1)
- added D1: LED_Right_Indicator(Yellow_LTH5MM12VFR4700), LED_THT:LED_D5.0mm, F.Cu at (186.6, 48.9)
- added D10: LED_2.2V_20ma, LED_THT:LED_D5.0mm, F.Cu at (130.9, 131.9)
- added D11: LED_2.2V_20ma, LED_THT:LED_D5.0mm, F.Cu at (123.4, 125.3)
- added D12: LED_2.2V_20ma, LED_THT:LED_D5.0mm, F.Cu at (118.5, 118.6)
- added D13: LED_2.2V_20ma, LED_THT:LED_D5.0mm, F.Cu at (114.9, 112.0)
- added D2: LED_High_Beam(Blue_LTH5MM12VFR4600), LED_THT:LED_D5.0mm, F.Cu at (176.2, 43.9)
- added D3: LED_Neutral(Green_LTH5MM12VFR4500), LED_THT:LED_D5.0mm, F.Cu at (145.3, 43.9)
- added D4: LED_Left_Indicator(Yellow_LTH5MM12VFR4700), LED_THT:LED_D5.0mm, F.Cu at (134.4, 49.0)
- added D5: LED_2.2V_20ma, LED_THT:LED_D5.0mm, F.Cu at (206.2, 112.0)
- added D7: LED_2.2V_20ma, LED_THT:LED_D5.0mm, F.Cu at (202.6, 118.6)
- added D8: LED_2.2V_20ma, LED_THT:LED_D5.0mm, F.Cu at (197.5, 125.3)
- added D9: LED_2.2V_20ma, LED_THT:LED_D5.0mm, F.Cu at (190.1, 131.9)
- added DS1: NHD-C12832A1Z-FS_RGB_-FBW-3V, Added_Footprints:NHDC12832A1ZFSRGBFBW3V, F.Cu at (148.5, 129.2)
- added H1: MountingHole, MountingHole:MountingHole_3.2mm_M3, F.Cu at (160.7, 140.2)
- added H2: MountingHole, MountingHole:MountingHole_3.2mm_M3, F.Cu at (202.4, 62.4)
- added H3: MountingHole, MountingHole:MountingHole_3.2mm_M3, F.Cu at (144.1, 52.7)
- added J2: Main_Power_In_JST-XH, Connector_JST:JST_XH_B2B-XH-A_1x02_P2.50mm_Vertical, B.Cu at (172.9, 49.3)
- added J3: Warning_Lights_JST-XH, Connector_JST:JST_XH_B4B-XH-A_1x04_P2.50mm_Vertical, B.Cu at (156.9, 40.8)
- added J4: Signals_RPM_Temp_Fuel_JST-XH, Connector_JST:JST_XH_B4B-XH-A_1x04_P2.50mm_Vertical, F.Cu at (125.9, 109.9)
- added J5: Speed_Pulser_Setup_Signal_JST-XH, Connector_Wire:SolderWirePad_1x01_SMD_1x2mm, B.Cu at (125.5, 52.6)
- added J6: Alphanumeric_Qwiick_JST-XH, Connector_JST:JST_XH_B4B-XH-A_1x04_P2.50mm_Vertical, F.Cu at (111.8, 103.4)
- added JP1: Pull up Jumper, Jumper:SolderJumper-3_P1.3mm_Open_RoundedPad1.0x1.5mm_NumberLabels, F.Cu at (109.5, 79.9)
- added M2: Stepper_Motor_bipolar, Added_Footprints:X27-168, F.Cu at (160.5, 84.3)
- added N1: Tachometer Reference, Added_Footprints:Dial_Gauge_Reference_CBF600, F.Cu at (160.5, 90.3)
- added R1: 200R, Resistor_SMD:R_0805_2012Metric_Pad1.20x1.40mm_HandSolder, F.Cu at (181.8, 44.1)
- added R10: 3.3KR, Resistor_SMD:R_0805_2012Metric_Pad1.20x1.40mm_HandSolder, F.Cu at (128.9, 75.3)
- added R11: 1KR, Resistor_SMD:R_0805_2012Metric_Pad1.20x1.40mm_HandSolder, F.Cu at (129.2, 70.7)
- added R12: 100R, Resistor_SMD:R_0805_2012Metric_Pad1.20x1.40mm_HandSolder, F.Cu at (194.6, 80.2)
- added R13: 100R, Resistor_SMD:R_0805_2012Metric_Pad1.20x1.40mm_HandSolder, F.Cu at (194.6, 82.8)
- added R14: 100R, Resistor_SMD:R_0805_2012Metric_Pad1.20x1.40mm_HandSolder, F.Cu at (194.5, 85.3)
- added R15: 100R, Resistor_SMD:R_0805_2012Metric_Pad1.20x1.40mm_HandSolder, F.Cu at (194.5, 87.8)
- added R16: 100R, Resistor_SMD:R_0805_2012Metric_Pad1.20x1.40mm_HandSolder, F.Cu at (194.5, 90.3)
- added R17: 100R, Resistor_SMD:R_0805_2012Metric_Pad1.20x1.40mm_HandSolder, F.Cu at (194.2, 92.8)
- added R18: 100R, Resistor_SMD:R_0805_2012Metric_Pad1.20x1.40mm_HandSolder, F.Cu at (194.2, 95.4)
- added R19: 100R, Resistor_SMD:R_0805_2012Metric_Pad1.20x1.40mm_HandSolder, F.Cu at (194.2, 97.9)
- added R2: 200R, Resistor_SMD:R_0805_2012Metric_Pad1.20x1.40mm_HandSolder, F.Cu at (169.1, 43.3)
- added R20: 10KR, Resistor_THT:R_Axial_DIN0204_L3.6mm_D1.6mm_P7.62mm_Horizontal, F.Cu at (107.5, 92.7)
- added R22: 56R, Resistor_SMD:R_0805_2012Metric_Pad1.20x1.40mm_HandSolder, B.Cu at (142.9, 121.4)
- added R23: 6.8R, Resistor_SMD:R_0805_2012Metric_Pad1.20x1.40mm_HandSolder, B.Cu at (174.8, 123.0)
- added R24: 6.8R, Resistor_SMD:R_0805_2012Metric_Pad1.20x1.40mm_HandSolder, B.Cu at (177.8, 123.0)
- added R25: 4.7KR, Resistor_SMD:R_0805_2012Metric_Pad1.20x1.40mm_HandSolder, F.Cu at (113.7, 80.4)
- added R26: 4.7KR, Resistor_SMD:R_0805_2012Metric_Pad1.20x1.40mm_HandSolder, F.Cu at (110.1, 74.9)
- added R3: 200R, Resistor_SMD:R_0805_2012Metric_Pad1.20x1.40mm_HandSolder, F.Cu at (152.9, 43.3)
- added R4: 200R, Resistor_SMD:R_0805_2012Metric_Pad1.20x1.40mm_HandSolder, F.Cu at (139.8, 43.6)
- added R5: 3.3KR, Resistor_SMD:R_0805_2012Metric_Pad1.20x1.40mm_HandSolder, F.Cu at (125.6, 64.9)
- added R6: 1KR, Resistor_SMD:R_0805_2012Metric_Pad1.20x1.40mm_HandSolder, F.Cu at (125.6, 70.6)
- added R7: 1KR, Resistor_SMD:R_0805_2012Metric_Pad1.20x1.40mm_HandSolder, F.Cu at (124.2, 95.6)
- added R8: 1KR, Resistor_SMD:R_0805_2012Metric_Pad1.20x1.40mm_HandSolder, F.Cu at (126.4, 91.7)
- added R9: 510R, Resistor_SMD:R_0805_2012Metric_Pad1.20x1.40mm_HandSolder, F.Cu at (128.7, 87.6)
- added SW1: SW_Push_JST-XH_Input, Connector_JST:JST_XH_B2B-XH-A_1x02_P2.50mm_Vertical, F.Cu at (112.5, 88.4)
- added TP1: TestPoint, Connector_PinHeader_1.00mm:PinHeader_1x01_P1.00mm_Vertical, B.Cu at (138.6, 66.7)
- added TP2: TestPoint, Connector_PinHeader_1.00mm:PinHeader_1x01_P1.00mm_Vertical, B.Cu at (117.0, 92.1)
- added TP3: TestPoint, Connector_PinHeader_1.00mm:PinHeader_1x01_P1.00mm_Vertical, B.Cu at (117.1, 66.8)
- added U1: R-78E3.3-0.5, Converter_DCDC:Converter_DCDC_RECOM_R-78E-0.5_THT, B.Cu at (206.8, 70.5)
- added U2: L293D, Package_DIP:DIP-16_W7.62mm, B.Cu at (156.8, 64.8)
- added U3: TEC2-1219WI, Converter_DCDC:Converter_DCDC_TRACO_TMR-xxxx_THT, B.Cu at (192.3, 56.6)
- added U4: L7805, Package_TO_SOT_THT:TO-220-3_Horizontal_TabDown, B.Cu at (184.9, 72.5)
- added U5: TXB0104D, Package_SO:SOIC-14_3.9x8.7mm_P1.27mm, B.Cu at (159.9, 79.7)
- added U6: 74HC595, Package_DIP:DIP-16_W7.62mm_Socket, B.Cu at (188.7, 82.7)
- added U7: CAT24C128, Package_SO:SOIC-8_3.9x4.9mm_P1.27mm, F.Cu at (114.2, 73.0)
Routing:
- net Net-(D12-A): track 0.00 -> 129.9 mm
- net Net-(D11-A): track 0.00 -> 129.7 mm
- net Net-(D13-A): track 0.00 -> 125.5 mm
- net Net-(D10-A): track 0.00 -> 125.4 mm
- net Net-(D9-A): track 0.00 -> 63.6 mm
- net Net-(D8-A): track 0.00 -> 58.7 mm
- net Net-(D7-A): track 0.00 -> 53.6 mm
- net Net-(D5-A): track 0.00 -> 49.4 mm
- net Net-(U2-2Y): track 0.00 -> 41.6 mm
- net Net-(U2-4Y): track 0.00 -> 31.5 mm
- net Net-(U2-3Y): track 0.00 -> 31.5 mm
- net Net-(U2-3A): track 0.00 -> 29.5 mm
- net Net-(U2-2A): track 0.00 -> 29.5 mm, vias 0 -> 1
- net Net-(M2--): track 0.00 -> 23.9 mm
- net Net-(U2-1A): track 0.00 -> 22.3 mm, vias 0 -> 1
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Other:
- board outline added: 110 x 110 mm

Commit message: Finished PCB layout for version 1
Parts:
- added C19: 0.1 uF, Capacitor_SMD:C_0805_2012Metric_Pad1.18x1.45mm_HandSolder, F.Cu at (118.4, 63.0)
- J4: moved to B.Cu
- TP1, TP2, TP3: footprint Connector_PinHeader_1.00mm:PinHeader_1x01_P1.00mm_Vertical -> Connector_PinHeader_2.54mm:PinHeader_1x01_P2.54mm_Vertical
- moved R7 5.43 mm to (126.1, 90.6)
- moved R8 5.02 mm to (128.4, 87.1)
- moved R9 4.76 mm to (131.3, 83.7)
- moved R10 3.70 mm to (132.5, 76.3), turned to 180 degrees
- moved R20 2.32 mm to (109.5, 91.6)
- moved TP1 2.08 mm to (140.7, 66.8)
- moved H3 1.98 mm to (145.7, 54.0)
- moved J5 1.89 mm to (126.7, 54.0)
- moved U7 1.51 mm to (115.7, 73.0)
- moved TP2 1.35 mm to (118.1, 92.8)
- moved A1 1.28 mm to (136.6, 61.6)
- moved C5 1.28 mm to (133.5, 70.7)
- moved R11 1.28 mm to (130.4, 70.7)
- moved C1 1.27 mm to (127.9, 60.6)
- moved R25 1.26 mm to (114.9, 80.5)
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Connections:
- A1 pad 12: /Data_Display_Controller/RES(RST) -> /Data_Display_Controller/SPI_CS(CS1B)
- A1 pad 13: /Data_Display_Controller/SPI_CS(CS1B) -> /Data_Display_Controller/RES(RST)
Routing:
- net /Data_Display_Controller/Bar_SER: track 0.00 -> 76.3 mm
- net /Data_Display_Controller/SPI_SCK: track 0.00 -> 75.9 mm
- net /Data_Display_Controller/Bar_RCLK: track 0.00 -> 73.2 mm
- net /Data_Display_Controller/Bar_SRCLK: track 0.00 -> 72.2 mm
- net /Data_Display_Controller/SPI_CS(CS1B): track 0.00 -> 62.9 mm
- net /Data_Display_Controller/RES(RST): track 0.00 -> 61.1 mm
- net /Data_Display_Controller/I2C SCL: track 0.00 -> 59.5 mm
- net /Data_Display_Controller/COPI(MOSI): track 0.00 -> 58.8 mm
- net /Data_Display_Controller/A0: track 0.00 -> 55.8 mm
- net /Data_Display_Controller/Tach_A1: track 0.00 -> 50.5 mm, vias 0 -> 1
- net /Data_Display_Controller/Tach_A2: track 0.00 -> 48.6 mm, vias 0 -> 1
- net /Data_Display_Controller/Tach_A3: track 0.00 -> 41.7 mm, vias 0 -> 1
- net /Data_Display_Controller/Tach_A4: track 0.00 -> 40.5 mm, vias 0 -> 1
- net Net-(J4-Pin_4): track 0.00 -> 37.7 mm
- net /Data_Display_Controller/I2C SDA: track 0.00 -> 37.5 mm
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- added copper zone on F.Cu, net +12V
- added copper zone on B.Cu, net +3.3V
- added copper zone on F.Cu, net +3.3V
- added copper zone on F.Cu, net +5V
- added copper zone on B.Cu, net +9V
- added copper zone on F.Cu, net +9V
- added copper zone on B.Cu, net GND
- added copper zone on F.Cu, net GND

Commit message: Slight modification to get more ground fill on the top layer to help with EMI
Routing:
- net GND: vias 10 -> 17
- net (no net): vias 1 -> 0
Changed lines of the file:
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@@
 		(layer "User.2")
-	)
-	(via
-		(at 245.618 73.533)
-		(size 0.8)
-		(drill 0.3)
-		(layers "F.Cu" "B.Cu")
-		(net 0)
 	)
 	(segment
@@
 	)
 	(via
+		(at 151.765 83.312)
+		(size 0.8)
+		(drill 0.3)
+		(layers "F.Cu" "B.Cu")
+		(free yes)
+		(net 4)
+	)
+	(via
 		(at 113.411 68.326)
 		(size 0.8)
@@
 	)
 	(via
+		(at 148.463 94.742)
+		(size 0.8)
+		(drill 0.3)
+		(layers "F.Cu" "B.Cu")
+		(free yes)
+		(net 4)
+	)
+	(via
 		(at 177.927 118.872)
 		(size 0.8)
@@
 	)
 	(via
+		(at 128.524 68.707)
+		(size 0.8)
+		(drill 0.3)
+		(layers "F.Cu" "B.Cu")
+		(free yes)
+		(net 4)
+	)
+	(via
+		(at 133.477 67.564)
+		(size 0.8)
+		(drill 0.3)
+		(layers "F.Cu" "B.Cu")
+		(free yes)
+		(net 4)
+	)
+	(via
 		(at 118.364 68.707)
 		(size 0.8)
@@
 	)
 	(via
+		(at 130.556 67.437)
+		(size 0.8)
+		(drill 0.3)
+		(layers "F.Cu" "B.Cu")
+		(free yes)
+		(net 4)
+	)
+	(via
+		(at 162.052 103.759)
+		(size 0.8)
+		(drill 0.3)
+		(layers "F.Cu" "B.Cu")
+		(free yes)
+		(net 4)
+	)
+	(via
 		(at 174.879 118.872)
 		(size 0.8)
@@
 		(size 0.8)
 		(drill 0.3)
+		(layers "F.Cu" "B.Cu")
+		(free yes)
+		(net 4)
+	)
+	(via
+		(at 131.318 60.579)
+		(size 0.8)
+		(drill 0.3)

Commit message: Slightly adjusted layout of board and made V1 gerbers. Generated PDF schematics
Routing:
- net Net-(D12-A): track 129.9 -> 121.4 mm
- net Net-(D11-A): track 129.7 -> 122.1 mm
- net Net-(D13-A): track 125.5 -> 120.0 mm
- net Net-(D7-A): track 53.6 -> 49.0 mm
- net Net-(D8-A): track 58.7 -> 54.1 mm
- net Net-(D10-A): track 125.4 -> 120.9 mm
- net Net-(D9-A): track 63.6 -> 59.1 mm
- net Net-(D5-A): track 49.4 -> 45.0 mm
- net /Data_Display_Controller/I2C SCL: track 59.5 -> 58.9 mm
- net GND: vias 17 -> 20
